File: CAD - Organizer/BSidesKC23_Organizer.kicad_pcb (KiCad board)
At the start: 2 copper layers, 54.8 x 147.9 mm, 75 parts, among them J1 UART, J2 JTAG, J3 Reset Jumper, J4 5v GND, J5 Boot Jumper, J6 USB, SW1 Boot, SW3 SW_Left, SW4 SW_Right, SW5 SW_Center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

Commit message: finishing up variants
Parts:
- removed the G*** at (53.6, 106.7)
- added G***: LOGO, BSidesKC:F.CU_OrgText, F.Cu at (53.5, 106.8)
- moved G*** 0.12 mm to (53.5, 106.8)
